File: lower_rear.sch (KiCad schematic (older format))
At the start: 3 parts, among them U6 CRIO, U7 WIFI_DC_CONV, U8 LIGHTS_DC_CONV

Commit message: Added more connector blocks and wire sizes
Connections:
- net CRIO_SOL_VIN: now reaches U6.21 (SVIN)
Changed lines of the file:
@@
 $Descr A4 11693 8268
 encoding utf-8
-Sheet 5 5
+Sheet 3 5
 Title ""
-Date "6 feb 2014"
+Date "7 feb 2014"
 Rev ""
 Comp ""
@@
 Wire Wire Line
 	1550 2850 2150 2850
+Text HLabel 4200 2650 2    60   Input ~ 12
+CRIO_SOL_VIN
+Wire Wire Line
+	3750 2650 4200 2650
 $EndSCHEMATC
