File: main_board.sch (KiCad schematic (older format))
At the start: 12 parts, among them U5 PD_BOARD

Commit message: Udpates to main board and start of connector spec.
Connections:
- net labels added: ELEV_VIN, INT_VIN, KICK_1_VIN, KICK_2_VIN, MOT_LB_VIN, MOT_LB_VOUT, MOT_LF_VIN, MOT_RB_VIN, MOT_RB_VOUT, MOT_RF_VIN, SPIKE_PWM
- net labels removed: MOT_LR_VOUT, MOT_RR_VOUT
- wire segments 123 -> 110
Other:
- note added: "20A"
- note added: "30A"
- note added: "5A"
Changed lines of the file:
@@
 $Descr A4 11693 8268
 encoding utf-8
-Sheet 3 5
+Sheet 5 5
 Title ""
 Date "6 feb 2014"
@@
 LIGHTS_VOUT
 Text HLabel 10150 1750 0    60   Output ~ 12
-MOT_RR_VOUT
+MOT_RB_VOUT
 Text HLabel 10350 850  0    60   Output ~ 12
 MOT_RF_VOUT
 Text HLabel 1750 3400 2    60   Output ~ 12
-MOT_LR_VOUT
+MOT_LB_VOUT
 Text HLabel 1700 2350 2    60   Output ~ 12
 MOT_LF_VOUT
@@
 	850  5850 850  2250
 Wire Wire Line
-	850  2250 8350 2250
-Wire Wire Line
-	8350 2250 8350 2550
-Wire Wire Line
-	8350 2550 9600 2550
+	850  2250 7050 2250
+Wire Wire Line
+	7050 2250 7050 2550
+Wire Wire Line
+	7050 2550 9600 2550
 Wire Wire Line
 	1450 5950 700  5950
@@
 	700  5950 700  2100
 Wire Wire Line
-	700  2100 8350 2100
-Wire Wire Line
-	8350 2100 8350 1600
-Wire Wire Line
-	8350 1600 9600 1600
+	700  2100 7050 2100
+Wire Wire Line
+	7050 2100 7050 1600
+Wire Wire Line
+	7050 1600 9600 1600
 Connection ~ 1450 5950
 Wire Wire Line
 	1300 6050 1300 4200
 Wire Wire Line
-	1300 4200 8350 4200
-Wire Wire Line
-	8350 4200 8350 4900
-Wire Wire Line
-	8350 4900 9600 4900
+	1300 4200 8200 4200
+Wire Wire Line
+	8200 4200 8200 4900
+Wire Wire Line
+	8200 4900 9600 4900
 Connection ~ 1450 6050
 Wire Wire Line
@@
 	1000 6150 1000 3200
 Wire Wire Line
-	1000 3200 8350 3200
-Wire Wire Line
-	8350 3200 8350 3850
-Wire Wire Line
-	8350 3850 9600 3850
+	1000 3200 8200 3200
+Wire Wire Line
+	8200 3200 8200 3850
+Wire Wire Line
+	8200 3850 9600 3850
 Wire Wire Line
 	1300 6050 1450 6050
@@
 Wire Wire Line
 	1400 1100 1400 1300
-Wire Wire Line
-	5000 5850 3500 5850
-Wire Wire Line
-	3500 5850 3500 2600
-Wire Wire Line
-	3500 2600 3000 2600
-Wire Wire Line
-	5000 5950 3400 5950
-Wire Wire Line
-	3400 5950 3400 3600
-Wire Wire Line
-	3400 3600 3000 3600
-Wire Wire Line
-	5000 6050 4950 6050
-Wire Wire Line
-	4950 6050 4950 4400
-Wire Wire Line
-	4950 4400 8800 4400
-Wire Wire Line
-	5000 6150 4900 6150
-Wire Wire Line
-	4900 6150 4900 3350
-Wire Wire Line
-	4900 3350 8800 3350
-Wire Wire Line
-	5000 6250 4850 6250
-Wire Wire Line
-	4850 6250 4850 2400
-Wire Wire Line
-	4850 2400 8700 2400
-Wire Wire Line
-	8700 2400 8700 2050
-Wire Wire Line
-	8700 2050 8800 2050
-Wire Wire Line
-	5000 6350 4800 6350
-Wire Wire Line
-	4800 6350 4800 1100
-Wire Wire Line
-	4800 1100 8800 1100
-Wire Wire Line
-	6750 5600 8250 5600
-Wire Wire Line
-	8250 5600 8250 1300
-Wire Wire Line
-	8250 1300 3000 1300
-Wire Wire Line
-	6750 5700 7000 5700
-Wire Wire Line
-	7000 5700 7000 4500
-Wire Wire Line
-	7000 4500 3000 4500
 Wire Wire Line
 	1450 6350 1100 6350
@@
 Wire Wire Line
 	3000 4800 3650 4800
-Text HLabel 3150 7450 2    60   Input ~ 12
+Text HLabel 3150 7450 2    60   Output ~ 12
 RSL_VOUT
 Wire Wire Line
@@
 Wire Wire Line
 	3100 6800 3550 6800
-Wire Wire Line
-	1250 6750 1450 6750
-Text HLabel 7250 5800 2    60   Input ~ 12
+Text HLabel 7250 5800 2    60   Output ~ 12
 CRIO_A_VOUT
 Wire Wire Line
@@
 Wire Wire Line
 	6850 3750 6500 3750
-Wire Wire Line
-	1250 6750 1250 7650
-Wire Wire Line
-	1250 7650 4500 7650
-Wire Wire Line
-	4500 7650 4500 3900
-Wire Wire Line
-	4500 3900 5300 3900
 Text HLabel 5300 3450 2    60   Output ~ 12
 COMP_VOUT+
@@
 Text Notes 6950 3550 0    60   ~ 12
 Note:\nCOMP_VOUT- comes from \nthe ground wire of the \nSpike relay's VIN wire.
+Text Notes 6700 5500 0    40   ~ 0
+20A
+Text Notes 6700 5400 0    40   ~ 0
+5A
+Text Notes 6700 5300 0    40   ~ 0
+5A
+Text Notes 6700 5600 0    40   ~ 0
+30A
+Text Notes 6700 5700 0    40   ~ 0
+30A
+Wire Wire Line
+	6750 5600 7200 5600
+Text Label 7200 5600 2    50   ~ 0
+INT_VIN
+Wire Wire Line
+	3000 1300 3350 1300
+Text Label 3350 1300 2    40   ~ 0
+INT_VIN
+Wire Wire Line
+	6750 5700 7200 5700
+Text Label 7200 5700 2    40   ~ 0
+ELEV_VIN
+Wire Wire Line
+	3000 4500 3500 4500
+Text Label 3500 4500 2    40   ~ 0
+ELEV_VIN
+Text Notes 6700 5800 0    40   ~ 0
+20A
+Text Notes 6700 5900 0    40   ~ 0
+20A
+Wire Wire Line
+	5300 3900 4900 3900
+Text Label 4900 3900 0    40   ~ 0
+SPIKE_PWM
+Wire Wire Line
+	1450 6750 1100 6750
+Text Label 1100 6750 2    40   ~ 0
+SPIKE_PWM
+Wire Wire Line
+	5000 5850 4500 5850
+Wire Wire Line
+	5000 5950 4500 5950
+Wire Wire Line
+	5000 6050 4500 6050
+Wire Wire Line
+	5000 6150 4500 6150
+Wire Wire Line
+	5000 6250 4500 6250
+Wire Wire Line
+	5000 6350 4500 6350
+Text Label 4500 5850 0    40   ~ 0
+MOT_RF_VIN
+Text Label 8300 1100 0    40   ~ 0
+MOT_RF_VIN
+Text Label 4500 5950 0    40   ~ 0
+MOT_RB_VIN
+Text Label 8300 2050 0    40   ~ 0
+MOT_RB_VIN
+Text Label 4500 6050 0    40   ~ 0
+MOT_LF_VIN
+Text Label 3450 2600 2    40   ~ 0
+MOT_LF_VIN
+Text Label 4500 6150 0    40   ~ 0
+MOT_LB_VIN
+Text Label 3500 3600 2    40   ~ 0
+MOT_LB_VIN
+Text Label 4500 6250 0    40   ~ 0
+KICK_1_VIN
+Text Label 8350 3350 0    40   ~ 0
+KICK_1_VIN
+Text Label 4500 6350 0    40   ~ 0
+KICK_2_VIN
+Text Label 8400 4400 0    40   ~ 0
+KICK_2_VIN
+Wire Wire Line
+	3000 2600 3450 2600
+Wire Wire Line
+	3000 3600 3500 3600
+Wire Wire Line
+	8800 1100 8300 1100
+Wire Wire Line
+	8800 2050 8300 2050
+Wire Wire Line
+	8800 3350 8350 3350
+Wire Wire Line
+	8800 4400 8400 4400
 $EndSCHEMATC

Commit message: Cleaned up main board schematic a little more
Connections:
- net labels added: DSC_VIN, ELEV_PWM, INT_PWM, KICK_1_PWM, KICK_2_PWM, MOT_LB_PWM, MOT_LF_PWM, MOT_RB_PWM, MOT_RF_PWM
- net labels removed: DSC_VOUT
- wire segments 110 -> 93
Other:
- note added: "Note:\nMake sure the Spike\nrelay has a 20A auto\nreset breaker."
- moved on the sheet: U?
Changed lines of the file:
@@
 Text HLabel 4350 5550 0    60   Output ~ 12
 WIFI_VOUT
-Text HLabel 7250 5300 2    60   Output ~ 12
+Text HLabel 7250 5400 2    60   Output ~ 12
 LIGHTS_VOUT
 Text HLabel 10150 1750 0    60   Output ~ 12
@@
 Text HLabel 1750 4300 2    60   Output ~ 12
 ELEV_VOUT
-Text HLabel 7250 5400 2    60   Output ~ 12
+Text HLabel 7250 5500 2    60   Output ~ 12
 CAM_LEDRING_VOUT
 Text HLabel 1700 1100 2    60   Output ~ 12
 INT_VOUT
-Text HLabel 7250 5500 2    60   Output ~ 12
-DSC_VOUT
 $Comp
 L TALON U?
@@
 L DIGITAL_SIDECAR U?
 U 1 1 52F325CA
-P 1200 5350
-F 0 "U?" H 2500 5200 60  0000 C CNN
-F 1 "DIGITAL_SIDECAR" H 2150 3100 60  0000 C CNN
-F 2 "~" H 1200 5350 60  0000 C CNN
-F 3 "~" H 1200 5350 60  0000 C CNN
-	1    1200 5350
+P 2150 6550
+F 0 "U?" H 3450 6400 60  0000 C CNN
+F 1 "DIGITAL_SIDECAR" H 3100 4300 60  0000 C CNN
+F 2 "~" H 2150 6550 60  0000 C CNN
+F 3 "~" H 2150 6550 60  0000 C CNN
+	1    2150 6550
 	1    0    0    -1
 $EndComp
@@
 	4350 5750 4600 5750
 Wire Wire Line
-	4350 5650 4600 5650
-Wire Wire Line
-	4600 5650 5000 5650
+	4350 5650 5000 5650
 Wire Wire Line
 	4350 5550 5000 5550
@@
 	4350 5200 5000 5200
 Wire Wire Line
-	7250 5500 6750 5500
+	7250 6200 6750 6200
+Wire Wire Line
+	6750 5500 7250 5500
 Wire Wire Line
 	6750 5400 7250 5400
 Wire Wire Line
-	6750 5300 7250 5300
-Wire Wire Line
 	9250 6000 8900 6000
 Wire Wire Line
@@
 	1400 4300 1750 4300
 Wire Wire Line
-	1450 5650 1200 5650
-Wire Wire Line
-	1200 5650 1200 3100
-Wire Wire Line
-	1450 5750 1150 5750
-Wire Wire Line
-	1150 5750 1150 4100
-Wire Wire Line
-	1150 4100 2200 4100
-Wire Wire Line
-	1450 5850 850  5850
-Wire Wire Line
-	850  5850 850  2250
-Wire Wire Line
-	850  2250 7050 2250
-Wire Wire Line
-	7050 2250 7050 2550
-Wire Wire Line
-	7050 2550 9600 2550
-Wire Wire Line
-	1450 5950 700  5950
-Wire Wire Line
-	700  5950 700  2100
-Wire Wire Line
-	700  2100 7050 2100
-Wire Wire Line
-	7050 2100 7050 1600
-Wire Wire Line
-	7050 1600 9600 1600
-Connection ~ 1450 5950
-Wire Wire Line
-	1300 6050 1300 4200
-Wire Wire Line
-	1300 4200 8200 4200
-Wire Wire Line
-	8200 4200 8200 4900
-Wire Wire Line
-	8200 4900 9600 4900
-Connection ~ 1450 6050
-Wire Wire Line
-	1450 6150 1000 6150
-Wire Wire Line
-	1000 6150 1000 3200
-Wire Wire Line
-	1000 3200 8200 3200
-Wire Wire Line
-	8200 3200 8200 3850
-Wire Wire Line
-	8200 3850 9600 3850
-Wire Wire Line
-	1300 6050 1450 6050
-Wire Wire Line
-	1450 6250 600  6250
-Wire Wire Line
-	600  6250 600  1800
-Wire Wire Line
-	600  1800 2200 1800
-Wire Wire Line
-	1200 3100 2200 3100
-Wire Wire Line
 	1400 3400 1400 3600
 Wire Wire Line
@@
 Wire Wire Line
 	1400 1100 1400 1300
-Wire Wire Line
-	1450 6350 1100 6350
-Wire Wire Line
-	1100 6350 1100 4800
-Wire Wire Line
-	1100 4800 1400 4800
 Text HLabel 3650 4700 2    60   Input ~ 12
 UP_LIM
@@
 Wire Wire Line
 	3000 4800 3650 4800
-Text HLabel 3150 7450 2    60   Output ~ 12
+Text HLabel 3150 7350 2    60   Output ~ 12
 RSL_VOUT
 Wire Wire Line
-	2850 7450 3150 7450
+	2850 7350 3150 7350
 Text HLabel 2300 5150 2    60   Input ~ 12
 DS_DB37
@@
 Wire Wire Line
 	3100 6800 3550 6800
-Text HLabel 7250 5800 2    60   Output ~ 12
+Text HLabel 7250 5600 2    60   Output ~ 12
 CRIO_A_VOUT
 Wire Wire Line
-	7250 5800 6750 5800
+	7250 5600 6750 5600
 $Comp
 L SPIKE_RELAY U?
@@
 $EndComp
 Wire Wire Line
-	6850 5900 6750 5900
-Wire Wire Line
-	6850 3450 6850 3750
-Wire Wire Line
-	6850 3750 6850 5900
-Wire Wire Line
-	6850 3750 6500 3750
+	6900 3450 6900 5300
+Wire Wire Line
+	6900 3750 6500 3750
 Text HLabel 5300 3450 2    60   Output ~ 12
 COMP_VOUT+
@@
 COMP_VOUT-
 Wire Wire Line
-	6800 3450 6850 3450
-Connection ~ 6850 3750
-Text Notes 6950 3550 0    60   ~ 12
+	6800 3450 6900 3450
+Text Notes 6950 3550 0    40   ~ 8
 Note:\nCOMP_VOUT- comes from \nthe ground wire of the \nSpike relay's VIN wire.
-Text Notes 6700 5500 0    40   ~ 0
+Text Notes 6750 6200 0    40   ~ 0
 20A
-Text Notes 6700 5400 0    40   ~ 0
+Text Notes 6800 5500 0    40   ~ 0
 5A
-Text Notes 6700 5300 0    40   ~ 0
+Text Notes 6800 5400 0    40   ~ 0
 5A
-Text Notes 6700 5600 0    40   ~ 0
+Text Notes 6750 6300 0    40   ~ 0
 30A
-Text Notes 6700 5700 0    40   ~ 0
+Text Notes 6750 6400 0    40   ~ 0
 30A
 Wire Wire Line
-	6750 5600 7200 5600
-Text Label 7200 5600 2    50   ~ 0
+	6750 6300 7250 6300
+Text Label 7250 6300 2    50   ~ 0
 INT_VIN
 Wire Wire Line
@@
 INT_VIN
 Wire Wire Line
-	6750 5700 7200 5700
-Text Label 7200 5700 2    40   ~ 0
+	6750 6400 7250 6400
+Text Label 7250 6400 2    40   ~ 0
 ELEV_VIN
 Wire Wire Line
@@
 Text Label 3500 4500 2    40   ~ 0
 ELEV_VIN
-Text Notes 6700 5800 0    40   ~ 0
+Text Notes 6750 5600 0    40   ~ 0
 20A
-Text Notes 6700 5900 0    40   ~ 0
+Text Notes 6750 5300 0    40   ~ 0
 20A
 Wire Wire Line
@@
 SPIKE_PWM
 Wire Wire Line
-	1450 6750 1100 6750
-Text Label 1100 6750 2    40   ~ 0
+	1450 6750 750  6750
+Text Label 750  6750 0    40   ~ 0
 SPIKE_PWM
 Wire Wire Line
@@
 Text Label 4500 6250 0    40   ~ 0
 KICK_1_VIN
-Text Label 8350 3350 0    40   ~ 0
+Text Label 8400 4400 0    40   ~ 0
 KICK_1_VIN
 Text Label 4500 6350 0    40   ~ 0
 KICK_2_VIN
-Text Label 8400 4400 0    40   ~ 0
+Text Label 8350 3350 0    40   ~ 0
 KICK_2_VIN
 Wire Wire Line
@@
 Wire Wire Line
 	8800 4400 8400 4400
+Text Label 750  5650 0    40   ~ 0
+MOT_LF_PWM
+Text Label 1300 3100 0    40   ~ 0
+MOT_LF_PWM
+Text Label 750  5750 0    40   ~ 0
+MOT_LB_PWM
+Text Label 1350 4100 0    40   ~ 0
+MOT_LB_PWM
+Text Label 750  5850 0    40   ~ 0
+MOT_RB_PWM
+Text Label 8300 2550 0    40   ~ 0
+MOT_RB_PWM
+Text Label 750  5950 0    40   ~ 0
+MOT_RF_PWM
+Text Label 8300 1600 0    40   ~ 0
+MOT_RF_PWM
+Text Label 8400 4900 0    40   ~ 0
+KICK_1_PWM
+Text Label 750  6150 0    40   ~ 0
+KICK_2_PWM
+Text Label 750  6050 0    40   ~ 0
+KICK_1_PWM
+Text Label 750  6250 0    40   ~ 0
+INT_PWM
+Text Label 1350 1800 0    40   ~ 0
+INT_PWM
+Text Label 750  6350 0    40   ~ 0
+ELEV_PWM
+Text Label 950  4800 0    40   ~ 0
+ELEV_PWM
+Wire Wire Line
+	1450 5650 750  5650
+Wire Wire Line
+	1450 5750 750  5750
+Wire Wire Line
+	1450 5850 750  5850
+Wire Wire Line
+	1450 5950 750  5950
+Wire Wire Line
+	1450 6050 750  6050
+Wire Wire Line
+	1450 6150 750  6150
+Wire Wire Line
+	1450 6250 750  6250
+Wire Wire Line
+	1450 6350 750  6350
+Wire Wire Line
+	1400 4800 950  4800
+Wire Wire Line
+	2200 4100 1350 4100
+Wire Wire Line
+	2200 3100 1300 3100
+Wire Wire Line
+	2200 1800 1350 1800
+Wire Wire Line
+	9600 1600 8300 1600
+Wire Wire Line
+	8300 2550 9600 2550
+Wire Wire Line
+	9600 3850 8350 3850
+Wire Wire Line
+	9600 4900 8400 4900
+Text Label 8350 3850 0    40   ~ 0
+KICK_2_PWM
+Wire Wire Line
+	6900 5300 6750 5300
+Connection ~ 6900 3750
+Text Notes 5750 4050 0    40   ~ 0
+Note:\nMake sure the Spike\nrelay has a 20A auto\nreset breaker.
+Text Label 7250 6200 2    40   ~ 0
+DSC_VIN
+Text Label 3150 7450 2    40   ~ 0
+DSC_VIN
+Wire Wire Line
+	2850 7450 3150 7450
 $EndSCHEMATC

Commit message: Added more connector blocks and wire sizes
Parts:
- gave numbers to parts that had none: 11
Connections:
- net labels added: KICK_LIMIT, RIGHT_ENC_A, RIGHT_ENC_B
- wire segments 93 -> 102
Changed lines of the file:
@@
 Sheet 5 5
 Title ""
-Date "6 feb 2014"
+Date "7 feb 2014"
 Rev ""
 Comp ""
@@
 INT_VOUT
 $Comp
-L TALON U?
+L TALON U17
 U 1 1 52F31FC7
 P 9600 2100
-F 0 "U?" H 10000 1900 60  0000 C CNN
+F 0 "U17" H 10000 1900 60  0000 C CNN
 F 1 "TALON" H 9250 1900 60  0000 C CNN
 F 2 "~" H 9050 2800 60  0000 C CNN
@@
 $EndComp
 $Comp
-L TALON U?
+L TALON U16
 U 1 1 52F31FDE
 P 9600 1150
-F 0 "U?" H 10000 950 60  0000 C CNN
+F 0 "U16" H 10000 950 60  0000 C CNN
 F 1 "TALON" H 9250 950 60  0000 C CNN
 F 2 "~" H 9050 1850 60  0000 C CNN
@@
 $EndComp
 $Comp
-L TALON U?
+L TALON U12
 U 1 1 52F31FE4
 P 2200 3650
-F 0 "U?" H 2600 3450 60  0000 C CNN
+F 0 "U12" H 2600 3450 60  0000 C CNN
 F 1 "TALON" H 1850 3450 60  0000 C CNN
 F 2 "~" H 1650 4350 60  0000 C CNN
@@
 $EndComp
 $Comp
-L TALON U?
+L TALON U11
 U 1 1 52F31FEA
 P 2200 2650
-F 0 "U?" H 2600 2450 60  0000 C CNN
+F 0 "U11" H 2600 2450 60  0000 C CNN
 F 1 "TALON" H 1850 2450 60  0000 C CNN
 F 2 "~" H 1650 3350 60  0000 C CNN
@@
 $EndComp
 $Comp
-L TALON U?
+L TALON U19
 U 1 1 52F31FF0
 P 9600 4450
-F 0 "U?" H 10000 4250 60  0000 C CNN
+F 0 "U19" H 10000 4250 60  0000 C CNN
 F 1 "TALON" H 9250 4250 60  0000 C CNN
 F 2 "~" H 9050 5150 60  0000 C CNN
@@
 $EndComp
 $Comp
-L TALON U?
+L TALON U18
 U 1 1 52F31FF6
 P 9600 3400
-F 0 "U?" H 10000 3200 60  0000 C CNN
+F 0 "U18" H 10000 3200 60  0000 C CNN
 F 1 "TALON" H 9250 3200 60  0000 C CNN
 F 2 "~" H 9050 4100 60  0000 C CNN
@@
 $EndComp
 $Comp
-L TALON U?
+L TALON U10
 U 1 1 52F32002
 P 2200 1350
-F 0 "U?" H 2600 1150 60  0000 C CNN
+F 0 "U10" H 2600 1150 60  0000 C CNN
 F 1 "TALON" H 1850 1150 60  0000 C CNN
 F 2 "~" H 1650 2050 60  0000 C CNN
@@
 $EndComp
 $Comp
-L JAGUAR U?
+L JAGUAR U13
 U 1 1 52F323B3
 P 2200 4650
-F 0 "U?" H 2600 4350 60  0000 C CNN
+F 0 "U13" H 2600 4350 60  0000 C CNN
 F 1 "JAGUAR" H 1900 4350 60  0000 C CNN
 F 2 "~" H 1650 5450 60  0000 C CNN
@@
 $EndComp
 $Comp
-L DIGITAL_SIDECAR U?
+L DIGITAL_SIDECAR U9
 U 1 1 52F325CA
 P 2150 6550
-F 0 "U?" H 3450 6400 60  0000 C CNN
+F 0 "U9" H 2100 5450 60  0000 C CNN
 F 1 "DIGITAL_SIDECAR" H 3100 4300 60  0000 C CNN
 F 2 "~" H 2150 6550 60  0000 C CNN
@@
 $EndComp
 $Comp
-L FPGA U?
+L FPGA U15
 U 1 1 52F325D9
 P 9250 5600
-F 0 "U?" H 10250 4950 60  0000 C CNN
+F 0 "U15" H 10250 4950 60  0000 C CNN
 F 1 "FPGA" H 9900 5750 60  0000 C CNN
 F 2 "~" H 9100 5800 60  0000 C CNN
@@
 Wire Wire Line
 	2150 5150 2300 5150
-Text HLabel 3550 6400 2    60   Input ~ 12
+Text HLabel 3550 6250 2    60   Input ~ 12
 LEFT_ENC_A
-Text HLabel 3550 6500 2    60   Input ~ 12
+Text HLabel 3550 6350 2    60   Input ~ 12
 LEFT_ENC_B
-Text HLabel 3550 6600 2    60   Input ~ 12
+Text HLabel 3550 6150 2    60   Input ~ 12
 COMP_SWITCH
-Text HLabel 3550 6700 2    60   Input ~ 12
+Text HLabel 3550 6650 2    60   Input ~ 12
 BELT_ENC_A
-Text HLabel 3550 6800 2    60   Input ~ 12
+Text HLabel 3550 6750 2    60   Input ~ 12
 BELT_ENC_B
-Wire Wire Line
-	2850 5650 3300 5650
-Wire Wire Line
-	3300 5650 3300 6400
-Wire Wire Line
-	3300 6400 3550 6400
-Wire Wire Line
-	2850 5750 3250 5750
-Wire Wire Line
-	3250 5750 3250 6500
-Wire Wire Line
-	3250 6500 3550 6500
-Wire Wire Line
-	2850 5850 3200 5850
-Wire Wire Line
-	3200 5850 3200 6600
-Wire Wire Line
-	3200 6600 3550 6600
-Wire Wire Line
-	2850 5950 3150 5950
-Wire Wire Line
-	3150 5950 3150 6700
-Wire Wire Line
-	3150 6700 3550 6700
-Wire Wire Line
-	2850 6050 3100 6050
-Wire Wire Line
-	3100 6050 3100 6800
-Wire Wire Line
-	3100 6800 3550 6800
 Text HLabel 7250 5600 2    60   Output ~ 12
 CRIO_A_VOUT
@@
 	7250 5600 6750 5600
 $Comp
-L SPIKE_RELAY U?
+L SPIKE_RELAY U14
 U 1 1 52F33917
 P 5900 3800
-F 0 "U?" H 6150 3600 60  0000 C CNN
+F 0 "U14" H 6150 3600 60  0000 C CNN
 F 1 "SPIKE_RELAY" H 5900 4000 60  0000 C CNN
 F 2 "~" H 5200 4150 60  0000 C CNN
@@
 Wire Wire Line
 	6750 6300 7250 6300
-Text Label 7250 6300 2    50   ~ 0
+Text Label 7250 6300 2    40   ~ 0
 INT_VIN
 Wire Wire Line
@@
 MOT_LB_PWM
 Text Label 750  5850 0    40   ~ 0
-MOT_RB_PWM
+MOT_RF_PWM
 Text Label 8300 2550 0    40   ~ 0
 MOT_RB_PWM
 Text Label 750  5950 0    40   ~ 0
-MOT_RF_PWM
+MOT_RB_PWM
 Text Label 8300 1600 0    40   ~ 0
 MOT_RF_PWM
@@
 Wire Wire Line
 	2850 7450 3150 7450
+Text HLabel 3550 6450 2    60   Input ~ 12
+RIGHT_ENC_A
+Text HLabel 3550 6550 2    60   Input ~ 12
+RIGHT_ENC_B
+Wire Wire Line
+	2850 5650 3350 5650
+Wire Wire Line
+	3350 5650 3350 6150
+Wire Wire Line
+	3350 6150 3550 6150
+Wire Wire Line
+	2850 5750 3300 5750
+Wire Wire Line
+	3300 5750 3300 6250
+Wire Wire Line
+	3300 6250 3550 6250
+Wire Wire Line
+	2850 5850 3250 5850
+Wire Wire Line
+	3250 5850 3250 6350
+Wire Wire Line
+	3250 6350 3550 6350
+Wire Wire Line
+	2850 5950 3200 5950
+Wire Wire Line
+	3200 5950 3200 6450
+Wire Wire Line
+	3200 6450 3550 6450
+Wire Wire Line
+	2850 6050 3150 6050
+Wire Wire Line
+	3150 6050 3150 6550
+Wire Wire Line
+	3150 6550 3550 6550
+Wire Wire Line
+	2850 6150 3100 6150
+Wire Wire Line
+	3100 6150 3100 6650
+Wire Wire Line
+	3100 6650 3550 6650
+Wire Wire Line
+	2850 6250 3050 6250
+Wire Wire Line
+	3050 6250 3050 6750
+Wire Wire Line
+	3050 6750 3550 6750
+Wire Wire Line
+	2850 6350 3000 6350
+Wire Wire Line
+	3000 6350 3000 6850
+Wire Wire Line
+	3000 6850 3550 6850
+Text HLabel 3550 6850 2    60   Input ~ 12
+KICK_LIMIT
 $EndSCHEMATC

Commit message: Modified layout of main board components.  Replaced more wires with net labels.
Connections:
- wire segments 102 -> 104
Other:
- moved on the sheet: U14, U15, U5, U9
